File: hovImuBoard.kicad_pcb (KiCad board)
At the start: 2 copper layers, 71.6 x 71.6 mm, 65 parts, among them J1 AVR-ISP-6, J2 Ext. Power, J3 54602-908LF, J4 AVR-JTAG-10, J5 ExtensionPort, J6 Debug, U1 LD2981, U2 BMX160, U3 SN65LVDS179DR, U4 ATmega1284P-AU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

Commit message: Conversion to KiCad 6.0, add 3D models
First commit after successful conversion.
Save first before cleanup of outdated KiCad 5 files. Just to be sure.

Added missing 3D models for various parts. Downloaded from SNAP-EDA or
directly from the manufacturer's site.
Parts:
- moved H1 0.11 mm to (133.7, 102.4)
Other:
- net class Default removed
- net class PWR2Pad removed
- net class Signal removed
