File: hovSerialAdapter/hovSerialAdapter.sch (KiCad schematic (older format))
At the start: 35 parts, among them J1 54602-908LF, J2 Barrel_Jack, J3 DB9_Female, J4 Ext. Power, J5 54602-908LF, U1 MAX3232, U2 SN65LVDS179DR, U3 TPS62172DSG

Commit message: Finalize design of serial adapter board V0.1
Add box symbol and footprint.
Finishing touches on the routings
Parts:
- removed LOGO2: Logo_Open_Hardware_Small, Symbol:OSHW-Symbol_6.7x6mm_Copper, symbol Graphic:Logo_Open_Hardware_Small
- added H1: Box, hovImuBoard:Box-MB655030, symbol hovImuBoard:Box
- added J6: RX, Connector_PinHeader_2.54mm:PinHeader_1x02_P2.54mm_Vertical, symbol Connector:Conn_01x02_Male
- added J7: TX, Connector_PinHeader_2.54mm:PinHeader_1x02_P2.54mm_Vertical, symbol Connector:Conn_01x02_Male
- J1, J5: DK_Detail_Page /product-detail/en/amphenol-icc-fci/54602-908LF/609-1046-ND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 -> (none); Family Modular Connectors - Jacks -> (none); Status Active -> (none)
- J2: value Barrel_Jack -> Power jack; footprint (none) -> hovImuBoard:CUI_PJ-036AH-SMT-TR; symbol Connector:Barrel_Jack -> Connector:Barrel_Jack_Switch; Description (none) -> CONN PWR JACK 2X5.5MM SOLDER; Digi-Key_PN (none) -> CP-036AHPJCT-ND; MPN (none) -> PJ-036AH-SMT-TR; Manufacturer (none) -> CUI Devices
- J3: Description (none) -> CONN DSUB RCPT 9POS SLDR CUP; Digi-Key_PN (none) -> L77SDE09S-ND; MPN (none) -> L77SDE09S; Manufacturer (none) -> Amphenol ICC (Commercial Products)
- LOGO1: footprint Symbol:OSHW-Symbol_6.7x6mm_Copper -> Symbol:OSHW-Symbol_6.7x6mm_SilkScreen
Connections:
- net +12V: now also U3.3 (EN)
- net GND: now also J2.3
- net RX: now also J6.2 (Pin_2); no longer U2.2 (R)
- net TX: now also J7.2 (Pin_2); no longer U2.3 (D)
- net TX_RS232: now reaches J3.2 (TXD), J5.4 (TX), U1.14 (T1OUT)
- net RX_RS232: now reaches J3.3 (RXD), J5.3 (RX), U1.13 (R1IN)
- new net RX_LVDS: J6.1 (Pin_1), U2.2 (R)
- new net TX_LVDS: J7.1 (Pin_1), U2.3 (D)
Changed lines of the file:
@@
 encoding utf-8
 Sheet 1 1
-Title "horOpenVario Serial converter for IMU board"
+Title "horOpenVario serial converter for IMU board"
 Date "12-Jul-2020"
 Rev "0.1"
@@
 	1    0    0    -1
 $EndComp
-Text Label 5100 3100 2    50   ~ 0
-RX
-Text Label 5100 3200 2    50   ~ 0
-TX
 Text Label 7100 3000 0    50   ~ 0
 RX+
@@
 F 0 "LOGO1" H 1750 1275 50  0001 C CNN
 F 1 "Logo_Open_Hardware_Small" H 1750 775 50  0001 C CNN
-F 2 "Symbol:OSHW-Symbol_6.7x6mm_Copper" H 1750 1000 50  0001 C CNN
+F 2 "Symbol:OSHW-Symbol_6.7x6mm_SilkScreen" H 1750 1000 50  0001 C CNN
 F 3 "~" H 1750 1000 50  0001 C CNN
 	1    1750 1000
-	1    0    0    -1
-$EndComp
-$Comp
-L Graphic:Logo_Open_Hardware_Small LOGO2
-U 1 1 5D5F6CFD
-P 2400 1000
-F 0 "LOGO2" H 2400 1275 50  0001 C CNN
-F 1 "Logo_Open_Hardware_Small" H 2400 775 50  0001 C CNN
-F 2 "Symbol:OSHW-Symbol_6.7x6mm_Copper" H 2400 1000 50  0001 C CNN
-F 3 "~" H 2400 1000 50  0001 C CNN
-	1    2400 1000
 	1    0    0    -1
 $EndComp
@@
 $EndComp
 Connection ~ 1950 6450
-Wire Wire Line
-	1950 6450 2300 6450
-$Comp
-L hovImuBoard:DB9_Female_RS-232-DCE J3
-U 1 1 5F115F9D
-P 1750 4150
-F 0 "J3" H 1930 4196 50  0000 L CNN
-F 1 "DB9_Female" H 1930 4105 50  0000 L CNN
-F 2 "Connector_Dsub:DSUB-9_Female_EdgeMount_P2.77mm" H 1750 4150 50  0001 C CNN
-F 3 " ~" H 1750 4150 50  0001 C CNN
-	1    1750 4150
-	-1   0    0    -1
-$EndComp
-$Comp
-L Connector:Barrel_Jack J2
+$Comp
+L Connector:Barrel_Jack_Switch J2
 U 1 1 5F15CF43
 P 1200 3200
 F 0 "J2" H 970 3158 50  0000 R CNN
-F 1 "Barrel_Jack" H 970 3249 50  0000 R CNN
-F 2 "" H 1250 3160 50  0001 C CNN
-F 3 "~" H 1250 3160 50  0001 C CNN
+F 1 "Power jack" H 970 3249 50  0000 R CNN
+F 2 "hovImuBoard:CUI_PJ-036AH-SMT-TR" H 1250 3160 50  0001 C CNN
+F 3 "https://www.cuidevices.com/product/resource/digikeypdf/pj-036ah-smt-tr.pdf" H 1250 3160 50  0001 C CNN
+F 4 "CONN PWR JACK 2X5.5MM SOLDER" H 1200 3200 50  0001 C CNN "Description"
+F 5 "CP-036AHPJCT-ND" H 1200 3200 50  0001 C CNN "Digi-Key_PN"
+F 6 "PJ-036AH-SMT-TR" H 1200 3200 50  0001 C CNN "MPN"
+F 7 "CUI Devices" H 1200 3200 50  0001 C CNN "Manufacturer"
 	1    1200 3200
 	1    0    0    -1
@@
 L power:GND #PWR012
 U 1 1 5F15DE42
-P 1500 3300
-F 0 "#PWR012" H 1500 3050 50  0001 C CNN
-F 1 "GND" H 1505 3127 50  0000 C CNN
-F 2 "" H 1500 3300 50  0001 C CNN
-F 3 "" H 1500 3300 50  0001 C CNN
-	1    1500 3300
+P 1650 3300
+F 0 "#PWR012" H 1650 3050 50  0001 C CNN
+F 1 "GND" H 1655 3127 50  0000 C CNN
+F 2 "" H 1650 3300 50  0001 C CNN
+F 3 "" H 1650 3300 50  0001 C CNN
+	1    1650 3300
 	0    -1   -1   0
 $EndComp
@@
 L power:+VDC #PWR011
 U 1 1 5F15EF68
-P 1500 3100
-F 0 "#PWR011" H 1500 3000 50  0001 C CNN
-F 1 "+VDC" H 1500 3375 50  0000 C CNN
-F 2 "" H 1500 3100 50  0001 C CNN
-F 3 "" H 1500 3100 50  0001 C CNN
-	1    1500 3100
+P 1650 3100
+F 0 "#PWR011" H 1650 3000 50  0001 C CNN
+F 1 "+VDC" H 1650 3375 50  0000 C CNN
+F 2 "" H 1650 3100 50  0001 C CNN
+F 3 "" H 1650 3100 50  0001 C CNN
+	1    1650 3100
 	0    1    1    0
 $EndComp
@@
 F 4 "609-1046-ND" H 1800 5850 60  0001 L CNN "Digi-Key_PN"
 F 5 "54602-908LF" H 1800 5950 60  0001 L CNN "MPN"
-F 6 "Modular Connectors - Jacks" H 1800 6150 60  0001 L CNN "Family"
-F 7 "/product-detail/en/amphenol-icc-fci/54602-908LF/609-1046-ND/1001360" H 1800 6350 60  0001 L CNN "DK_Detail_Page"
-F 8 "CONN MOD JACK 8P8C R/A UNSHLD" H 1800 6450 60  0001 L CNN "Description"
-F 9 "Amphenol ICC (FCI)" H 1800 6550 60  0001 L CNN "Manufacturer"
-F 10 "Active" H 1800 6650 60  0001 L CNN "Status"
+F 6 "CONN MOD JACK 8P8C R/A UNSHLD" H 1800 6450 60  0001 L CNN "Description"
+F 7 "Amphenol ICC (FCI)" H 1800 6550 60  0001 L CNN "Manufacturer"
 	1    1600 5450
 	0    1    -1   0
@@
 F 4 "609-1046-ND" H 8950 3400 60  0001 L CNN "Digi-Key_PN"
 F 5 "54602-908LF" H 8950 3500 60  0001 L CNN "MPN"
-F 6 "Modular Connectors - Jacks" H 8950 3700 60  0001 L CNN "Family"
-F 7 "/product-detail/en/amphenol-icc-fci/54602-908LF/609-1046-ND/1001360" H 8950 3900 60  0001 L CNN "DK_Detail_Page"
-F 8 "CONN MOD JACK 8P8C R/A UNSHLD" H 8950 4000 60  0001 L CNN "Description"
-F 9 "Amphenol ICC (FCI)" H 8950 4100 60  0001 L CNN "Manufacturer"
-F 10 "Active" H 8950 4200 60  0001 L CNN "Status"
+F 6 "CONN MOD JACK 8P8C R/A UNSHLD" H 8950 4000 60  0001 L CNN "Description"
+F 7 "Amphenol ICC (FCI)" H 8950 4100 60  0001 L CNN "Manufacturer"
 	1    8750 3000
 	0    -1   1    0
@@
 Connection ~ 2300 3950
 Wire Wire Line
-	2300 3950 2300 3100
-Wire Wire Line
 	2050 4150 2400 4150
-Wire Wire Line
-	2400 3500 2400 4150
-Connection ~ 2400 4150
 Wire Wire Line
 	2400 4150 2400 5550
@@
 	1    0    0    -1
 $EndComp
-Wire Wire Line
-	4150 3500 4650 3500
-Wire Wire Line
-	4650 3500 4650 3200
 $Comp
 L power:GND #PWR04
@@
 Wire Wire Line
 	8350 3200 8100 3200
-Wire Wire Line
-	4650 3200 5100 3200
-Wire Wire Line
-	4150 3100 5100 3100
 $Comp
 L Interface_UART:MAX3232 U1
@@
 	1    0    0    -1
 $EndComp
+$Comp
+L power:PWR_FLAG #FLG0101
+U 1 1 5F135F8C
+P 7450 1300
+F 0 "#FLG0101" H 7450 1375 50  0001 C CNN
+F 1 "PWR_FLAG" H 7450 1473 50  0000 C CNN
+F 2 "" H 7450 1300 50  0001 C CNN
+F 3 "~" H 7450 1300 50  0001 C CNN
+	1    7450 1300
+	1    0    0    -1
+$EndComp
+Wire Wire Line
+	2250 6550 2250 6450
+Wire Wire Line
+	1950 6450 2250 6450
+Connection ~ 2250 6450
+Wire Wire Line
+	2250 6450 2300 6450
+Wire Wire Line
+	1500 3100 1650 3100
+Wire Wire Line
+	1500 3300 1650 3300
+Wire Wire Line
+	1500 3200 1500 3300
+Connection ~ 1500 3300
+Connection ~ 2400 4150
+Wire Wire Line
+	2400 3500 2400 4150
+Wire Wire Line
+	2300 3950 2300 3100
+$Comp
+L hovImuBoard:DB9_Female_RS-232-DCE J3
+U 1 1 5F115F9D
+P 1750 4150
+F 0 "J3" H 1930 4196 50  0000 L CNN
+F 1 "DB9_Female" H 1930 4105 50  0000 L CNN
+F 2 "Connector_Dsub:DSUB-9_Female_EdgeMount_P2.77mm" H 1750 4150 50  0001 C CNN
+F 3 "https://cdn.amphenol-icc.com/media/wysiwyg/files/documentation/datasheet/cmio/sd_hd_stamepd_formed_solder_cup_dsub.pdf" H 1750 4150 50  0001 C CNN
+F 4 "CONN DSUB RCPT 9POS SLDR CUP" H 1750 4150 50  0001 C CNN "Description"
+F 5 "L77SDE09S-ND" H 1750 4150 50  0001 C CNN "Digi-Key_PN"
+F 6 "L77SDE09S" H 1750 4150 50  0001 C CNN "MPN"
+F 7 "Amphenol ICC (Commercial Products)" H 1750 4150 50  0001 C CNN "Manufacturer"
+	1    1750 4150
+	-1   0    0    -1
+$EndComp
+$Comp
+L Connector:Conn_01x02_Male J6
+U 1 1 5F17A14F
+P 4400 3650
+F 0 "J6" V 4500 3500 50  0000 C CNN
+F 1 "RX" V 4350 3600 50  0000 C CNN
+F 2 "Connector_PinHeader_2.54mm:PinHeader_1x02_P2.54mm_Vertical" H 4400 3650 50  0001 C CNN
+F 3 "~" H 4400 3650 50  0001 C CNN
+F 4 "PinHeader1x02 P2.54mm Vertical" H 4400 3650 50  0001 C CNN "Description"
+	1    4400 3650
+	1    0    0    -1
+$EndComp
+$Comp
+L Connector:Conn_01x02_Male J7
+U 1 1 5F17FE08
+P 5000 3650
+F 0 "J7" V 5100 3500 50  0000 C CNN
+F 1 "TX" V 4950 3600 50  0000 C CNN
+F 2 "Connector_PinHeader_2.54mm:PinHeader_1x02_P2.54mm_Vertical" H 5000 3650 50  0001 C CNN
+F 3 "~" H 5000 3650 50  0001 C CNN
+F 4 "PinHeader1x02 P2.54mm Vertical" H 5000 3650 50  0001 C CNN "Description"
+	1    5000 3650
+	-1   0    0    -1
+$EndComp
+Text Label 5100 3100 2    50   ~ 0
+RX_LVDS
+Text Label 5100 3200 2    50   ~ 0
+TX_LVDS
+Text Label 4650 3650 1    50   ~ 0
+RX_LVDS
+Text Label 4650 3750 3    50   ~ 0
+RX
+Wire Wire Line
+	4600 3650 4650 3650
+Wire Wire Line
+	4600 3750 4650 3750
+Text Label 4150 3100 0    50   ~ 0
+RX
+Text Label 4150 3500 0    50   ~ 0
+TX
+Text Label 4800 3750 3    50   ~ 0
+TX
+Text Label 4800 3650 1    50   ~ 0
+TX_LVDS
+Text Label 2400 4150 0    50   ~ 0
+RX_RS232
+Text Label 2300 3950 0    50   ~ 0
+TX_RS232
+$Comp
+L hovImuBoard:Box H1
+U 1 1 5F1C2B5C
+P 9550 1450
+F 0 "H1" H 9550 1825 50  0000 C CNN
+F 1 "Box" H 9550 1734 50  0000 C CNN
+F 2 "hovImuBoard:Box-MB655030" H 9550 1450 50  0001 C CNN
+F 3 "https://www.hammfg.com/part/MB655030" H 9550 1450 50  0001 C CNN
+F 4 "BOX PLASTIC GRAY 2.56\"L X 1.97\"W" H 9550 1450 50  0001 C CNN "Description"
+F 5 "HM5530-ND" H 9550 1450 50  0001 C CNN "Digi-Key_PN"
+F 6 "MB655030" H 9550 1450 50  0001 C CNN "MPN"
+F 7 "Hammond Manufacturing" H 9550 1450 50  0001 C CNN "Manufacturer"
+	1    9550 1450
+	1    0    0    -1
+$EndComp

Commit message: hovSerialAdapter: Add 3D models from SnapEDA.
Add 3D models from SnapEDA to the footprints of the RJ-45 jack, and for the 8.2uH inductivity
Parts:
- L4: footprint Inductor_SMD:L_1812_4532Metric -> hovImuBoard:IND_LQH43PH8R2M26L; Description FIXED IND 8.2UH 1.3A 128 MOHM -> FIXED IND 8.2UH 1.3A 153.6 MOHM; Digi-Key_PN 490-16860-1-ND -> 490-16115-1-ND; MPN LQH43PN8R2M26L -> LQH43PH8R2M26L
Changed lines of the file:
@@
 F 0 "L4" V 4140 5050 50  0000 C CNN
 F 1 "8.2uH" V 4049 5050 50  0000 C CNN
-F 2 "Inductor_SMD:L_1812_4532Metric" H 3950 5050 50  0001 C CNN
-F 3 "https://search.murata.co.jp/Ceramy/image/img/P02/JELF243A-0093.pdf" H 3950 5050 50  0001 C CNN
-F 4 "490-16860-1-ND" H 3950 5050 50  0001 C CNN "Digi-Key_PN"
-F 5 "LQH43PN8R2M26L" H 3950 5050 50  0001 C CNN "MPN"
+F 2 "hovImuBoard:IND_LQH43PH8R2M26L" H 3950 5050 50  0001 C CNN
+F 3 "https://search.murata.co.jp/Ceramy/image/img/P02/JELF243A-9137.pdf" H 3950 5050 50  0001 C CNN
+F 4 "490-16115-1-ND" H 3950 5050 50  0001 C CNN "Digi-Key_PN"
+F 5 "LQH43PH8R2M26L" H 3950 5050 50  0001 C CNN "MPN"
 F 6 "Murata Electronics" H 3950 5050 50  0001 C CNN "Manufacturer"
-F 7 "FIXED IND 8.2UH 1.3A 128 MOHM" H 3950 5050 50  0001 C CNN "Description"
+F 7 "FIXED IND 8.2UH 1.3A 153.6 MOHM" H 3950 5050 50  0001 C CNN "Description"
 	1    3950 5050
 	0    -1   -1   0

Commit message: hovSerialAdapter: Add 3D model for the D-Sub connector.
Copy the footprint to lib/hovImuBoard.pretty, and add the 3D model.
Improve the switching trace on the 3.3V regulator, moving the feedback further out of the way
Parts:
- J3: footprint Connector_Dsub:DSUB-9_Female_EdgeMount_P2.77mm -> hovImuBoard:DSUB-9_Female_EdgeMount_P2.77mm
Changed lines of the file:
@@
 F 0 "J3" H 1930 4196 50  0000 L CNN
 F 1 "DB9_Female" H 1930 4105 50  0000 L CNN
-F 2 "Connector_Dsub:DSUB-9_Female_EdgeMount_P2.77mm" H 1750 4150 50  0001 C CNN
+F 2 "hovImuBoard:DSUB-9_Female_EdgeMount_P2.77mm" H 1750 4150 50  0001 C CNN
 F 3 "https://cdn.amphenol-icc.com/media/wysiwyg/files/documentation/datasheet/cmio/sd_hd_stamepd_formed_solder_cup_dsub.pdf" H 1750 4150 50  0001 C CNN
 F 4 "CONN DSUB RCPT 9POS SLDR CUP" H 1750 4150 50  0001 C CNN "Description"
